File: Implementering/Vuggesystem/Kredsløb/v1.0/MotorController.sch (EAGLE design)
At the start: 27 parts, among them Q1 IRF512, Q2 IRF512, Q3 IRF512, Q4 IRF512

Commit message: har lavet print til motor kreds, og lavet lidt på motor kontrol -Felix
Parts:
- removed Q1, Q2, Q3, Q4: IRF512, transistor-power:IRF512
- removed X3: (no value), con-wago-500:W237-4
- added C7, C8: 1.2pF, SparkFun-Passives:CAPPTH1
- added IC1: 74HC08N, 74xx-eu:74HC08N
- added IC2: 74HC04N, 74xx-eu:74HC04N
- added R10: 3.3 kOhm, rcl:R-EU_0207/10
- added U$1, U$2, U$3, U$4: IRFZ24N, transistor-power:IRFZ24N
- R9: value 10 Ohm -> 3.3 kOhm
- SV1: device con-lstb:MA05-1 -> con-lstb:MA03-1
Connections:
- removed net ES_SIG: R9.1, SV1.4, X3-1.KL, X3-3.KL
- new net N$10: IC1B.I0, IC2A.I, IC2B.O, R10.1
- new net N$15: C7.1, IC1A.I0, R9.2
- new net N$16: C8.1, IC1B.I1, R10.2
- new net PWM: IC1A.I1, IC2A.O, IC2B.I, R9.1, SV1.2
- net +3V3: now also IC2C.I, IC2D.I, IC2E.I, IC2F.I, SV1.3; no longer R9.2, SV1.5
- net GND: now also C7.2, C8.2, IC1C.I0, IC1C.I1, IC1D.I0, IC1D.I1, U$2.S, U$4.S; no longer Q2.S, Q3.S, X3-2.KL, X3-4.KL
- net MOT_A: now also U$1.S, U$4.D; no longer Q1.S, Q2.D
- net MOT_B: now also U$2.D, U$3.S; no longer Q3.D, Q4.S
- net M_A: now also IC1A.O; no longer SV1.3
- net M_B: now also IC1B.O; no longer SV1.2
- net N$3: now also U$1.G; no longer Q1.G
- net N$4: now also U$4.G; no longer Q2.G
- net N$5: now also U$3.G; no longer Q4.G
- net N$6: now also U$2.G; no longer Q3.G
- net VCC: now also U$1.D, U$3.D; no longer Q1.D, Q4.D
Other:
- note added: "Dead-time kreds"
- note added: "Ubrugte elementer"
- moved on the sheet: R9, X1-1, X1-2
