File: Implementering/Vuggesystem/Kredsløb/MotorController.brd (EAGLE design)
At the start: 75.9 x 82.5 mm, 27 parts, among them Q1 IRF512, Q2 IRF512, Q3 IRF512, Q4 IRF512

Commit message: VS: tilføjet optokobler afsnit -Felix
Parts:
- added OK1, OK2: HCPL2200, optocoupler:DIL08
- added R10, R11: 620 Ohm, rcl:0207/10
- moved SV1 56.5 mm to (9.53, 76.2), turned to 270 degrees
- moved R9 47.3 mm to (19.1, 74.9)
- moved SV2 3.81 mm to (5.08, 77.5), turned to 90 degrees
- moved C3 2.22 mm to (38.1, 46.0)
Connections:
- new net AGND: OK1.3, OK2.3, SV1.1, SV2.2, SV2.4
- new net N$10: OK1.2, R10.2
- new net N$11: OK2.2, R11.2
- new net N$14: OK2.5, OK2.6
- new net N$16: OK1.5, OK1.6
- new net PWM: R10.1, SV1.3
- new net PWM_N: R11.1, SV1.2
- net GND: no longer SV1.1, SV2.2, SV2.4
- net M_A: now also IO2.3, OK1.7; no longer IO1.3, SV1.2
- net M_B: now also IO1.3, OK2.7; no longer IO2.3, SV1.3
Routing:
- net AGND: track 0.00 -> 72.1 mm
- net M_B: track 18.6 -> 70.4 mm
- net ES_SIG: track 67.1 -> 18.1 mm
- net N$11: track 0.00 -> 46.3 mm
- net N$10: track 0.00 -> 42.5 mm
- net GND: track 41.7 -> 7.68 mm
- net +3V3: track 2.54 -> 16.2 mm
- net N$7: track 317.5 -> 327.7 mm
- net N$1: track 317.5 -> 327.7 mm
- net PWM_N: track 0.00 -> 4.97 mm
- net PWM: track 0.00 -> 4.97 mm
- net M_A: track 59.3 -> 55.0 mm
- net N$16: track 0.00 -> 2.54 mm
- net N$14: track 0.00 -> 2.54 mm
Other:
- board size 75.9 x 82.5 mm -> 75.9 x 87.6 mm
